File: PD_Regulation/PD_Regulation.kicad_sch (KiCad schematic)
At the start: 21 parts, among them J1 ADC Out, J2 TC Out, J3 LC Out, J4 Stepper Out, U1 uA7810, U2 L7805, U3 LD1086D2T33TR

Commit message: Completed PCB for PD board
Parts:
- removed C1, C3: 0.33μF, symbol Device:C_Small
- removed C10, C16, C8: 22μF, symbol Device:C_Small
- removed C5, C6: 10μF, symbol Device:C_Small
- removed J4: Stepper Out, TerminalBlock:TerminalBlock_Xinya_XY308-2.54-2P_1x02_P2.54mm_Horizontal, symbol Connector:Screw_Terminal_01x02
- added C1, C11, C13, C5, C7, C9: 10μF, Capacitor_THT:CP_Radial_D5.0mm_P2.00mm, symbol Device:C_Polarized_Small_US
- added C2: 0.1μF, Capacitor_THT:C_Disc_D4.7mm_W2.5mm_P5.00mm, symbol Device:C_Small
- added J4: GND, TerminalBlock:TerminalBlock_Xinya_XY308-2.54-5P_1x05_P2.54mm_Horizontal, symbol Connector:Screw_Terminal_01x05
- added J5: 24V Out, TerminalBlock:TerminalBlock_Xinya_XY308-2.54-5P_1x05_P2.54mm_Horizontal, symbol Connector:Screw_Terminal_01x05
- added J6: 24VIN, TerminalBlock:TerminalBlock_Xinya_XY308-2.54-2P_1x02_P2.54mm_Horizontal, symbol Connector:Screw_Terminal_01x02
- C10: renamed from C11; footprint (none) -> Capacitor_THT:C_Disc_D4.7mm_W2.5mm_P5.00mm
- C12: value 22μF -> 0.1μF; footprint (none) -> Capacitor_THT:C_Disc_D4.7mm_W2.5mm_P5.00mm
- C14: renamed from C15; footprint (none) -> Capacitor_THT:C_Disc_D4.7mm_W2.5mm_P5.00mm
- C3: renamed from C2; footprint (none) -> Capacitor_THT:C_Disc_D4.7mm_W2.5mm_P5.00mm
- C4: footprint (none) -> Capacitor_THT:C_Disc_D4.7mm_W2.5mm_P5.00mm
- C6: renamed from C9; footprint (none) -> Capacitor_THT:C_Disc_D4.7mm_W2.5mm_P5.00mm
- C8: renamed from C7; footprint (none) -> Capacitor_THT:C_Disc_D4.7mm_W2.5mm_P5.00mm
Connections:
- net +10V: now also C11.1; no longer C10.1, J2.1 (Pin_1), J3.2 (Pin_2)
- net +24V: now also C1.1, C13.1, C2.1, J5.1 (Pin_1), J5.2 (Pin_2), J5.3 (Pin_3), J5.4 (Pin_4), J5.5 (Pin_5), J6.2 (Pin_2)
- net +3.3V: now also C5.1
- net +5V: now also C10.1, J2.1 (Pin_1), J3.2 (Pin_2), C7.1, C9.1
- net GND: now also C1.2, C11.2, C13.2, C2.2, C5.2, C7.2, C9.2, J4.1 (Pin_1), J4.2 (Pin_2), J4.3 (Pin_3), J4.4 (Pin_4), J4.5 (Pin_5), J6.1 (Pin_1)
Other:
- moved on the sheet: C14, C3, C4, U1, U2, U3
