File: PD_Regulation/PD_Regulation.kicad_pcb (KiCad board)
At the start: 2 copper layers, 7 parts, among them J1 ADC Out, J2 TC Out, J3 LC Out, J4 Stepper Out, U1 uA7810, U2 L7805, U3 LD1086D2T33TR

Commit message: Completed PCB for PD board
Parts:
- added C1: 10μF, Capacitor_THT:CP_Radial_D5.0mm_P2.00mm, F.Cu at (84.0, 92.5)
- added C10: 0.1μF, Capacitor_THT:C_Disc_D4.7mm_W2.5mm_P5.00mm, F.Cu at (138.0, 95.5)
- added C11: 10μF, Capacitor_THT:CP_Radial_D5.0mm_P2.00mm, F.Cu at (119.5, 91.5)
- added C12: 0.1μF, Capacitor_THT:C_Disc_D4.7mm_W2.5mm_P5.00mm, F.Cu at (128.5, 95.5)
- added C13: 10μF, Capacitor_THT:CP_Radial_D5.0mm_P2.00mm, F.Cu at (92.0, 96.0)
- added C14: 0.1μF, Capacitor_THT:C_Disc_D4.7mm_W2.5mm_P5.00mm, F.Cu at (96.5, 96.5)
- added C2: 0.1μF, Capacitor_THT:C_Disc_D4.7mm_W2.5mm_P5.00mm, F.Cu at (84.0, 88.0)
- added C3: 0.1μF, Capacitor_THT:C_Disc_D4.7mm_W2.5mm_P5.00mm, F.Cu at (95.0, 83.6)
- added C4: 0.1μF, Capacitor_THT:C_Disc_D4.7mm_W2.5mm_P5.00mm, F.Cu at (111.3, 83.6)
- added C5: 10μF, Capacitor_THT:CP_Radial_D5.0mm_P2.00mm, F.Cu at (128.0, 71.0)
- added C6: 0.1μF, Capacitor_THT:C_Disc_D4.7mm_W2.5mm_P5.00mm, F.Cu at (129.5, 76.0)
- added C7: 10μF, Capacitor_THT:CP_Radial_D5.0mm_P2.00mm, F.Cu at (128.5, 87.0)
- added C8: 0.1μF, Capacitor_THT:C_Disc_D4.7mm_W2.5mm_P5.00mm, F.Cu at (137.5, 83.5)
- added C9: 10μF, Capacitor_THT:CP_Radial_D5.0mm_P2.00mm, F.Cu at (135.5, 91.5)
- added H1: MountingHole, MountingHole:MountingHole_3.2mm_M3_DIN965, F.Cu at (106.5, 93.5)
- added H1: MountingHole, MountingHole:MountingHole_3.2mm_M3_DIN965, F.Cu at (95.0, 66.5)
- added H1: MountingHole, MountingHole:MountingHole_3.2mm_M3_DIN965, F.Cu at (136.5, 66.0)
- added J5: 24V Out, TerminalBlock:TerminalBlock_Xinya_XY308-2.54-5P_1x05_P2.54mm_Horizontal, F.Cu at (101.5, 102.5)
- added J6: 24VIN, TerminalBlock:TerminalBlock_Xinya_XY308-2.54-2P_1x02_P2.54mm_Horizontal, F.Cu at (82.8, 101.8)
- J4: value Stepper Out -> GND; footprint TerminalBlock:TerminalBlock_Xinya_XY308-2.54-2P_1x02_P2.54mm_Horizontal -> TerminalBlock:TerminalBlock_Xinya_XY308-2.54-5P_1x05_P2.54mm_Horizontal
- moved J4 76.5 mm to (116.2, 102.5), turned to 180 degrees
- moved J3 61.6 mm to (128.5, 102.5), turned to 180 degrees
- moved J1 55.6 mm to (134.5, 78.5), turned to 90 degrees
- moved J2 53.2 mm to (137.0, 102.5), turned to 180 degrees
- moved U3 29.8 mm to (119.3, 75.9)
- moved U2 24.7 mm to (103.3, 75.9)
- moved U1 23.2 mm to (86.8, 75.7)
Connections:
- J2 pad 1: +10V -> +5V
- J3 pad 2: +10V -> +5V
- J4 pad 1: +24V -> GND
Routing:
- net +5V: track 0.00 -> 88.5 mm
- net +10V: track 0.00 -> 62.8 mm
- net +24V: track 0.00 -> 51.9 mm
- net +3.3V: track 0.00 -> 17.0 mm
- added copper zone on B.Cu, net GND
- added copper zone on F.Cu, net GND
Other:
- board outline added: 61 x 44 mm
- board text added: "24V"
- board text added: "24VIN"
- board text added: "24VOUT"
- board text added: "5 3.3 GND"
- board text added: "ADC"
- board text added: "GND"
- board text added: "GND 5"
- board text added: "GND GND 5 10"
- board text added: "LC"
- board text added: "QRET Power Distribution"
- board text added: "TC"

Commit message: Added vias
Parts:
- moved H1 1.03 mm to (106.2, 94.5)
- moved H1 0.50 mm to (95.0, 66.0)
Routing:
- net GND: vias 0 -> 20
Other:
- board text added: "L7805"
- board text added: "LD1086D2T33TR"
- board text added: "uA7810"
